File: studies/console/hardware/field_buttons_2025/keyboard.kicad_pcb (KiCad board)
At the start: 2 copper layers, 289.5 x 169.5 mm, 69 parts, among them J1 Conn_02x12_Counter_Clockwise, SW1 SW_Push, SW10 SW_Push, SW11 SW_Push, SW12 SW_Push, SW13 SW_Push, SW14 SW_Push, SW15 SW_Push, SW16 SW_Push, SW17 SW_Push, SW18 SW_Push, SW19 SW_Push, SW2 SW_Push, SW20 SW_Push, SW21 SW_Push, SW22 SW_Push, SW23 SW_Push, SW24 SW_Push, SW25 SW_Push, SW26 SW_Push, SW27 SW_Push, SW28 SW_Push, SW29 SW_Push, SW3 SW_Push, SW30 SW_Push, SW31 SW_Push, SW32 SW_Push, SW4 SW_Push, SW5 SW_Push, SW6 SW_Push, SW7 SW_Push, SW8 SW_Push, SW9 SW_Push

Commit message: i added microcontroller tracks and code
Parts:
- D1, D10, D11, D12, D13, D14, D15, D16, D17, D18, D19, D2, D20, D22, D23, D24, D25, D26, D27, D28, D29, D3, D30, D31, D32, D4, D6, D7, D8, D9: moved to F.Cu
- moved D1 92.1 mm to (136.5, 73.5)
- moved SW1 92.1 mm to (125.0, 68.5)
- moved D2 82.4 mm to (192.8, 73.5)
- moved SW2 82.1 mm to (181.0, 68.5)
- moved J1 75.2 mm to (100.5, 139.2)
- moved D3 72.3 mm to (248.5, 73.5)
- moved SW3 72.3 mm to (237.0, 68.5)
- moved H2 65.2 mm to (345.0, 68.5)
- moved D32 63.6 mm to (356.9, 208.5)
- moved SW32 63.2 mm to (345.0, 203.5)
- moved SW4 62.7 mm to (293.0, 68.5)
- moved SW23 62.6 mm to (258.1, 168.5)
- moved D15 62.6 mm to (171.1, 130.7)
- moved D17 62.6 mm to (236.8, 150.6)
- moved D10 62.6 mm to (314.4, 116.6)
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Connections:
- J1 pad 10: unconnected-(J1-Pin_10-Pad10) -> /COL3
- J1 pad 11: unconnected-(J1-Pin_11-Pad11) -> /COL2
- J1 pad 12: unconnected-(J1-Pin_12-Pad12) -> /COL1
- J1 pad 13: unconnected-(J1-Pin_13-Pad13) -> /ROW4
- J1 pad 14: unconnected-(J1-Pin_14-Pad14) -> /ROW3
- J1 pad 15: unconnected-(J1-Pin_15-Pad15) -> /ROW2
- J1 pad 16: unconnected-(J1-Pin_16-Pad16) -> /ROW1
- J1 pad 17: unconnected-(J1-Pin_17-Pad17) -> /ROW0
- J1 pad 6: unconnected-(J1-Pin_6-Pad6) -> /COL0
- J1 pad 7: unconnected-(J1-Pin_7-Pad7) -> /COL6
- J1 pad 8: unconnected-(J1-Pin_8-Pad8) -> /COL5
- J1 pad 9: unconnected-(J1-Pin_9-Pad9) -> /COL4
Routing:
- net /COL6: track 213.3 -> 506.0 mm
- net /COL5: track 229.5 -> 474.8 mm
- net /COL4: track 184.9 -> 408.7 mm
- net /COL3: track 221.2 -> 364.5 mm
- net /COL2: track 111.0 -> 247.5 mm
- net /COL1: track 210.4 -> 320.6 mm
- net /ROW0: track 313.1 -> 418.3 mm
- net /ROW1: track 205.0 -> 292.3 mm
- net /ROW4: track 289.6 -> 373.2 mm
- net /ROW2: track 174.9 -> 247.0 mm
- net /ROW3: track 196.0 -> 248.0 mm
- net /COL0: track 155.6 -> 172.7 mm
- net Net-(D7-A): track 8.95 -> 6.68 mm
- net Net-(D32-A): track 8.88 -> 9.42 mm
Other:
- board size 289.5 x 169.5 mm -> 311 x 174 mm

Commit message: add logo and strain relief
Parts:
- added G***: LOGO, Graphics:wildhat_logo_6_med, F.Cu at (136.5, 203.0)
- added REF**: MountingHole_3.2mm_M3_ISO7380_Pad, MountingHole:MountingHole_3.2mm_M3_ISO7380_Pad, F.Cu at (88.5, 112.5)
- added REF**: MountingHole_3.2mm_M3_ISO7380_Pad, MountingHole:MountingHole_3.2mm_M3_ISO7380_Pad, F.Cu at (95.0, 112.5)
- added REF**: MountingHole_3.2mm_M3_ISO7380_Pad, MountingHole:MountingHole_3.2mm_M3_ISO7380_Pad, F.Cu at (95.0, 68.5)
- added REF**: MountingHole_3.2mm_M3_ISO7380_Pad, MountingHole:MountingHole_3.2mm_M3_ISO7380_Pad, F.Cu at (88.5, 68.5)
- moved J1 19.9 mm to (84.5, 151.0)
- moved D7 1.80 mm to (154.0, 101.6)
- moved D6 0.08 mm to (119.2, 101.6)
Connections:
- J1 pad 10: /COL3 -> /COL4
- J1 pad 11: /COL2 -> /COL5
- J1 pad 12: /COL1 -> /COL6
- J1 pad 7: /COL6 -> /COL1
- J1 pad 8: /COL5 -> /COL2
- J1 pad 9: /COL4 -> /COL3
Routing:
- net /COL6: track 506.0 -> 470.4 mm
- net /COL5: track 474.8 -> 446.6 mm
- net /ROW0: track 418.3 -> 442.4 mm
- net /ROW1: track 292.3 -> 314.9 mm
- net /COL4: track 408.7 -> 387.2 mm
- net /ROW2: track 247.0 -> 267.9 mm
- net /COL3: track 364.5 -> 350.3 mm
- net /ROW3: track 248.0 -> 259.4 mm
- net /COL0: track 172.7 -> 179.1 mm
- net /COL2: track 247.5 -> 241.2 mm
- net /ROW4: track 373.2 -> 377.9 mm
- net Net-(D7-A): track 6.68 -> 8.48 mm
- net /COL1: track 320.6 -> 322.0 mm
Other:
- board text added: "Jan 20, 2025"
- board text removed: "100"
