File: studies/console/hardware/field_buttons_2025/keyboard.kicad_pcb (KiCad board)
At the start: 2 copper layers, 311 x 174 mm, 74 parts, among them J1 Conn_02x12_Counter_Clockwise, SW1 SW_Push, SW10 SW_Push, SW11 SW_Push, SW12 SW_Push, SW13 SW_Push, SW14 SW_Push, SW15 SW_Push, SW16 SW_Push, SW17 SW_Push, SW18 SW_Push, SW19 SW_Push, SW2 SW_Push, SW20 SW_Push, SW21 SW_Push, SW22 SW_Push, SW23 SW_Push, SW24 SW_Push, SW25 SW_Push, SW26 SW_Push, SW27 SW_Push, SW28 SW_Push, SW29 SW_Push, SW3 SW_Push, SW30 SW_Push, SW31 SW_Push, SW32 SW_Push, SW4 SW_Push, SW5 SW_Push, SW6 SW_Push, SW7 SW_Push, SW8 SW_Push, SW9 SW_Push

Commit message: move logo, shrink board a little
Parts:
- moved G*** 164.4 mm to (245.0, 79.5)
Other:
- board size 311 x 174 mm -> 305 x 168 mm
Changed lines of the file:
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@@
 	(footprint "Graphics:wildhat_logo_6_med"
 		(layer "F.Cu")
-		(at 136.5 203)
+		(at 245 79.5)
 		(property "Reference" "G***"
 			(at 0 0 0)
@@
 	)
 	(gr_line
-		(start 365 49.97912)
-		(end 365 224)
+		(start 361.5 52)
+		(end 361.5 220)
 		(stroke
 			(width 0.4)
@@
 	)
 	(gr_line
-		(start 54 224)
-		(end 54 50)
+		(start 56.5 220)
+		(end 56.5 52)
 		(stroke
 			(width 0.4)
@@
 	)
 	(gr_line
-		(start 365 224)
-		(end 54 224)
+		(start 361.5 220)
+		(end 56.5 220)
 		(stroke
 			(width 0.4)
@@
 	)
 	(gr_line
-		(start 54 50)
-		(end 365 49.97912)
+		(start 56.5 52)
+		(end 361.5 52)
 		(stroke
 			(width 0.4)
@@
 	)
 	(gr_text "Jan 20, 2025"
-		(at 252 222 0)
+		(at 101.5 213 0)
 		(layer "F.SilkS")
 		(effects

Commit message: use round-number inches for holes and outline
Parts:
- moved H4 4.11 mm to (346.2, 181.4)
- moved H3 4.11 mm to (71.8, 181.4)
- moved H2 1.79 mm to (346.2, 67.1)
- moved H1 1.79 mm to (71.8, 67.1)
- renumbered REF** to H5, REF** to H6, REF** to H7, REF** to H8
Other:
- board size 305 x 168 mm -> 304.8 x 165.1 mm
- board text added: "Jan 23, 2025"
- board text removed: "Jan 20, 2025"
Changed lines of the file:
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@@
 	(footprint "MountingHole:MountingHole_4.3mm_M4_ISO7380_Pad"
 		(layer "F.Cu")
-		(at 345 177.5)
+		(at 346.16 181.44)
 		(descr "Mounting Hole 4.3mm, M4, ISO7380")
 		(tags "mounting hole 4.3mm m4 iso7380")
@@
 	(footprint "MountingHole:MountingHole_4.3mm_M4_ISO7380_Pad"
 		(layer "F.Cu")
-		(at 73 177.5)
+		(at 71.84 181.44)
 		(descr "Mounting Hole 4.3mm, M4, ISO7380")
 		(tags "mounting hole 4.3mm m4 iso7380")
@@
 	(footprint "MountingHole:MountingHole_4.3mm_M4_ISO7380_Pad"
 		(layer "F.Cu")
-		(at 345 68.5)
+		(at 346.16 67.14)
 		(descr "Mounting Hole 4.3mm, M4, ISO7380")
 		(tags "mounting hole 4.3mm m4 iso7380")
@@
 		(descr "Mounting Hole 3.2mm, M3, ISO7380")
 		(tags "mounting hole 3.2mm m3 iso7380")
-		(property "Reference" "REF**"
+		(property "Reference" "H7"
 			(at 0 -3.85 0)
 			(layer "F.SilkS")
@@
 		(descr "Mounting Hole 3.2mm, M3, ISO7380")
 		(tags "mounting hole 3.2mm m3 iso7380")
-		(property "Reference" "REF**"
+		(property "Reference" "H8"
 			(at 0 -3.85 0)
 			(layer "F.SilkS")
@@
 	(footprint "MountingHole:MountingHole_4.3mm_M4_ISO7380_Pad"
 		(layer "F.Cu")
-		(at 73 68.5)
+		(at 71.84 67.14)
 		(descr "Mounting Hole 4.3mm, M4, ISO7380")
 		(tags "mounting hole 4.3mm m4 iso7380")
@@
 		(descr "Mounting Hole 3.2mm, M3, ISO7380")
 		(tags "mounting hole 3.2mm m3 iso7380")
-		(property "Reference" "REF**"
+		(property "Reference" "H6"
 			(at 0 -3.85 0)
 			(layer "F.SilkS")
@@
 		(descr "Mounting Hole 3.2mm, M3, ISO7380")
 		(tags "mounting hole 3.2mm m3 iso7380")
-		(property "Reference" "REF**"
+		(property "Reference" "H5"
 			(at 0 -3.85 0)
 			(layer "F.SilkS")
@@
 	)
 	(gr_line
-		(start 361.5 52)
-		(end 361.5 220)
+		(start 361.4 54.44)
+		(end 361.4 219.54)
 		(stroke
 			(width 0.4)
@@
 	)
 	(gr_line
-		(start 56.5 220)
-		(end 56.5 52)
+		(start 56.6 219.54)
+		(end 56.6 54.44)
 		(stroke
 			(width 0.4)
@@
 	)
 	(gr_line
-		(start 361.5 220)
-		(end 56.5 220)
+		(start 361.4 219.54)
+		(end 56.6 219.54)
 		(stroke
 			(width 0.4)
@@
 	)
 	(gr_line
-		(start 56.5 52)
-		(end 361.5 52)
+		(start 56.6 54.44)
+		(end 361.4 54.44)
 		(stroke
 			(width 0.4)
@@
 		(layer "Edge.Cuts")
 	)
-	(gr_text "Jan 20, 2025"
+	(gr_text "Jan 23, 2025"
 		(at 101.5 213 0)
 		(layer "F.SilkS")
